File: Genesis Numpad.kicad_pcb (KiCad board)
At the start: 2 copper layers, 107.2 x 123 mm, 56 parts, among them SW1 SW_Push, U1 ATmega32U4-AU, Y1 16MHz

Commit message: Fixed Errors in design
Parts:
- moved R4 3.27 mm to (133.3, 31.0), turned to 180 degrees
- moved C1 2.38 mm to (123.0, 23.0)
- moved C5 1.84 mm to (122.9, 44.7)
- moved C2 1.59 mm to (133.3, 34.1)
Routing:
- net +5V: track 125.6 -> 130.2 mm
- net COL3: track 221.1 -> 223.9 mm
- net COL1: track 264.4 -> 267.1 mm
- net COL0: track 285.7 -> 288.3 mm
- net COL2: track 242.9 -> 244.9 mm
- net Net-(R4-Pad2): track 6.01 -> 4.07 mm
- net GND: track 36.4 -> 37.5 mm
