File: _autosave-Genesis Numpad.kicad_pcb (KiCad board)
At the start: 2 copper layers, 107.2 x 123 mm, 56 parts, among them SW1 SW_Push, U1 ATmega32U4-AU, Y1 16MHz

Commit message: Adjusted traces
Routing:
- net +5V: track 96.9 -> 65.8 mm
- net GND: track 50.6 -> 45.5 mm, vias 4 -> 0
Changed lines of the file:
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@@
     (thickness 1.6)
     (drawings 17)
-    (tracks 476)
+    (tracks 459)
     (zones 0)
     (modules 56)
@@
   (segment (start 124.233332 24.537166) (end 124.550249 24.220249) (width 0.381) (layer B.Cu) (net 1))
   (segment (start 124.233332 27.272314) (end 124.233332 24.537166) (width 0.381) (layer B.Cu) (net 1))
-  (segment (start 119.566427 38.727444) (end 120.65 37.643871) (width 0.381) (layer B.Cu) (net 1))
-  (segment (start 129.3245 35.899017) (end 128.350483 34.925) (width 0.381) (layer B.Cu) (net 1))
   (segment (start 117.86937 31.232112) (end 118.418979 31.781721) (width 0.381) (layer B.Cu) (net 1))
-  (via (at 124.61875 35.71875) (size 0.8) (drill 0.4) (layers F.Cu B.Cu) (net 1))
   (segment (start 124.249408 36.088092) (end 124.61875 35.71875) (width 0.381) (layer B.Cu) (net 1))
-  (segment (start 124.249408 39.874891) (end 124.249408 36.088092) (width 0.381) (layer B.Cu) (net 1))
   (segment (start 124.799017 40.4245) (end 124.249408 39.874891) (width 0.381) (layer B.Cu) (net 1))
-  (segment (start 124.61875 35.71875) (end 124.61875 32.54375) (width 0.381) (layer F.Cu) (net 1))
-  (via (at 124.61875 32.54375) (size 0.8) (drill 0.4) (layers F.Cu B.Cu) (net 1))
-  (via (at 120.65 32.54375) (size 0.8) (drill 0.4) (layers F.Cu B.Cu) (net 1))
-  (segment (start 124.61875 32.54375) (end 120.65 32.54375) (width 0.381) (layer F.Cu) (net 1))
-  (via (at 120.904 37.211) (size 0.8) (drill 0.4) (layers F.Cu B.Cu) (net 1))
-  (segment (start 120.65 36.957) (end 120.904 37.211) (width 0.381) (layer F.Cu) (net 1))
-  (segment (start 120.65 32.54375) (end 120.65 36.957) (width 0.381) (layer F.Cu) (net 1))
   (segment (start 117.86937 31.232112) (end 117.846112 31.232112) (width 0.381) (layer B.Cu) (net 1))
   (segment (start 117.846112 31.232112) (end 116.967 30.353) (width 0.381) (layer B.Cu) (net 1))
@@
   (segment (start 134.14375 35.71875) (end 134.14375 34.925) (width 0.381) (layer B.Cu) (net 1))
   (segment (start 124.233332 27.272314) (end 124.233332 27.372918) (width 0.381) (layer B.Cu) (net 1))
-  (segment (start 124.233332 27.372918) (end 123.03125 28.575) (width 0.381) (layer B.Cu) (net 1))
+  (segment (start 129.3245 35.899017) (end 128.350483 34.925) (width 0.381) (layer B.Cu) (net 1))
+  (segment (start 124.249408 39.874891) (end 124.202891 39.874891) (width 0.381) (layer B.Cu) (net 1))
+  (segment (start 124.202891 39.874891) (end 123.444 39.116) (width 0.381) (layer B.Cu) (net 1))
+  (segment (start 119.566427 38.727444) (end 119.641556 38.727444) (width 0.381) (layer B.Cu) (net 1))
+  (segment (start 122.552353 38.177836) (end 124.799017 40.4245) (width 0.381) (layer B.Cu) (net 1))
+  (segment (start 120.191164 38.177836) (end 122.552353 38.177836) (width 0.381) (layer B.Cu) (net 1))
+  (segment (start 119.641556 38.727444) (end 120.191164 38.177836) (width 0.381) (layer B.Cu) (net 1))
+  (segment (start 125.4125 34.925) (end 124.249408 36.088092) (width 0.381) (layer B.Cu) (net 1))
+  (segment (start 128.350483 34.925) (end 125.4125 34.925) (width 0.381) (layer B.Cu) (net 1))
+  (segment (start 124.799017 40.4245) (end 124.799017 40.471017) (width 0.381) (layer B.Cu) (net 1))
+  (segment (start 124.799017 40.471017) (end 125.984 41.656) (width 0.381) (layer B.Cu) (net 1))
   (segment (start 125.893751 26.743266) (end 125.893751 25.563751) (width 0.381) (layer B.Cu) (net 2))
   (segment (start 124.799017 27.838) (end 125.893751 26.743266) (width 0.381) (layer B.Cu) (net 2))
@@
   (segment (start 130.080103 35.523249) (end 129.890186 35.333332) (width 0.381) (layer B.Cu) (net 2))
   (segment (start 132.424249 35.523249) (end 130.080103 35.523249) (width 0.381) (layer B.Cu) (net 2))
-  (segment (start 122.2375 30.399517) (end 124.799017 27.838) (width 0.381) (layer B.Cu) (net 2))
-  (segment (start 122.2375 33.793629) (end 122.2375 30.399517) (width 0.381) (layer B.Cu) (net 2))
-  (segment (start 128.350483 33.793629) (end 122.2375 33.793629) (width 0.381) (layer B.Cu) (net 2))
-  (segment (start 129.890186 35.333332) (end 128.350483 33.793629) (width 0.381) (layer B.Cu) (net 2))
-  (segment (start 121.813091 39.874892) (end 121.263483 40.4245) (width 0.381) (layer B.Cu) (net 2))
-  (segment (start 124.233332 40.990186) (end 123.118038 39.874892) (width 0.381) (layer B.Cu) (net 2))
-  (segment (start 122.843858 39.874892) (end 122.2375 39.268534) (width 0.381) (layer B.Cu) (net 2))
-  (segment (start 123.118038 39.874892) (end 122.843858 39.874892) (width 0.381) (layer B.Cu) (net 2))
-  (segment (start 122.843858 39.874892) (end 121.813091 39.874892) (width 0.381) (layer B.Cu) (net 2))
-  (segment (start 122.2375 35.71875) (end 121.27494 34.75619) (width 0.381) (layer B.Cu) (net 2))
-  (segment (start 122.2375 39.268534) (end 122.2375 35.71875) (width 0.381) (layer B.Cu) (net 2))
-  (segment (start 121.27494 34.75619) (end 122.2375 33.793629) (width 0.381) (layer B.Cu) (net 2))
-  (segment (start 119.417564 36.613564) (end 119.417564 36.359564) (width 0.381) (layer B.Cu) (net 2))
-  (segment (start 118.435056 37.596073) (end 119.417564 36.613564) (width 0.381) (layer B.Cu) (net 2))
-  (segment (start 119.417564 36.613564) (end 121.27494 34.75619) (width 0.381) (layer B.Cu) (net 2))
-  (segment (start 119.417564 36.359564) (end 117.983 34.925) (width 0.381) (layer B.Cu) (net 2))
-  (segment (start 117.983 32.477113) (end 117.303685 31.797798) (width 0.381) (layer B.Cu) (net 2))
-  (segment (start 117.983 34.925) (end 117.983 32.477113) (width 0.381) (layer B.Cu) (net 2))
+  (segment (start 122.588269 42.635249) (end 120.232249 42.635249) (width 0.381) (layer B.Cu) (net 2))
+  (segment (start 124.233332 40.990186) (end 122.588269 42.635249) (width 0.381) (layer B.Cu) (net 2))
   (segment (start 117.104002 25.8445) (end 117.0305 25.8445) (width 0.25) (layer B.Cu) (net 3))
   (segment (start 119.035751 23.912751) (end 117.104002 25.8445) (width 0.25) (layer B.Cu) (net 3))
